Commit message: Adds velocity smoother

File: cultureid_turtlebot_description/robots/turtlebot_one_camera.urdf.xacro (robot description, xacro)
@@ -20,5 +20,5 @@
   <xacro:property name="M_PI" value="3.1415926535897931" />
   <xacro:sensor_orbbec_astra prefix="front_rgbd_camera" parent="base_link" prefix_topic="front_rgbd_camera">
-    <origin xyz="0.13 0.0 0.3148" rpy="0 0 0"/>
+    <origin xyz="0.1024 0.0 0.8808" rpy="0 0 0"/>
   </xacro:sensor_orbbec_astra>
   <kobuki/>

File: cultureid_turtlebot_description/turtlebot/urdf/turtlebot_properties.urdf.xacro (robot description, xacro)
@@ -21,5 +21,5 @@
 	<xacro:property name="cam_px" value="0.1024" />
 <!--	<xacro:property name="cam_py" value="-0.0125" /> Y varies for different configurations. get sets in sensors_urdf -->
-	<xacro:property name="cam_pz" value="0.2870" />
+	<xacro:property name="cam_pz" value="0.8808" />
 	<xacro:property name="cam_or" value="0" />
 	<xacro:property name="cam_op" value="0" />
