Commit message: Can function with num_cameras=0

File: cultureid_turtlebot_description/robots/turtlebot_zero_cameras.urdf.xacro (robot description, xacro)
@@ -4,5 +4,5 @@
     - Stacks    : hexagons
     - 2d Sensor : rplidar (or hokuyo)
-    - 3d Sensor : astra
+    - 3d Sensor : none
     - imu       : imu
 -->
@@ -11,5 +11,4 @@
   <xacro:include filename="$(find cultureid_turtlebot_description)/kobuki/urdf/kobuki.urdf.xacro" />
   <xacro:include filename="$(find cultureid_turtlebot_description)/turtlebot/urdf/stacks/hexagons.urdf.xacro"/>
-  <xacro:include filename="$(find cultureid_turtlebot_description)/turtlebot/urdf/sensors/orbbec_astra.urdf.xacro"/>
   <xacro:include filename="$(find cultureid_turtlebot_description)/turtlebot/urdf/sensors/ydlidar_tg30.urdf.xacro"/>
   <!--
@@ -18,8 +17,4 @@
   <xacro:include filename="$(find cultureid_turtlebot_description)/turtlebot/urdf/sensors/imu.urdf.xacro"/>
   -->
-  <xacro:property name="M_PI" value="3.1415926535897931" />
-  <xacro:sensor_orbbec_astra prefix="front_rgbd_camera" parent="base_link" prefix_topic="front_rgbd_camera">
-    <origin xyz="0.0424 0.0 0.8808" rpy="0 0 0"/>
-  </xacro:sensor_orbbec_astra>
   <kobuki/>
   <stack_hexagons parent="base_link"/>
